File: PLA/pla_xc9536.sch (EAGLE design)
At the start: 5 parts

Commit message: updated schematic to remove floating pins
Parts:
- removed JP2: (no value), pinhead-new:PINHD-2X3M
- added SJ1, SJ2, SJ3, SJ4: (no value), jumper:SJ2W
Connections:
- removed net N$1: CPLDG.GCK0, JP2.2
- removed net N$2: CPLDG.GCK1, JP2.4
- removed net N$3: CPLDG.GCK2, JP2.6
- removed net N$4: CPLDG.GTS0, JP2.1
- removed net N$5: CPLDG.GSR, JP2.5
- removed net N$6: CPLDG.FB1MC1, JP2.3
- new net 1: CPLDG.GCK0, SJ1.2
- new net 2: CPLDG.GCK1, SJ2.2
- new net 3: CPLDG.FB1MC1, SJ3.2
- new net 4: CPLDG.GTS0, SJ4.2
- net GND: now also CPLDG.FB2MC1, CPLDG.FB2MC2, CPLDG.GCK2, CPLDG.GSR, CPLDG.GTS1, SJ1.1, SJ2.1, SJ3.1, SJ4.1
- net PLA1: now also CPLDG.FB2MC7
- net TCK: now also JP1.3; no longer JP1.4
- net TMS: now also JP1.4; no longer JP1.3
- net VCC: now also SJ1.3, SJ2.3, SJ3.3, SJ4.3
